Commit message: URDF file for Gazebo simulation

File: urdf/model.urdf.xacro (robot description, xacro)
@@ -11,5 +11,5 @@
 	<xacro:property name = "elbow_width" value = "0.02"/>
 	<xacro:property name = "elbow_height" value = "0.05"/>
-	<xacro:property name = "elbow_length" value = "0.10"/>
+	<xacro:property name = "elbow_length" value = "0.15"/>
 	<link name = "world"/>
 	<link name = "base_link">
@@ -73,17 +73,23 @@
 			</inertial>
 		<visual name = "elbow_link_visual">
-			<origin xyz = "${base_radius} 0 ${-mount_length}" />
+			<origin xyz = "${-mount_width/2} ${mount_length} 0" />
 			<geometry>
 				<box size = "${elbow_width} ${elbow_length} ${elbow_height}"/>
 			</geometry>
 		</visual>
-		<visual name = "second_elbow_link">
-			<origin xyz = "${base_radius} ${base_radius} ${-mount_height}"/>
+		<visual name = "second_elbow_link_visual">
+			<origin xyz = "${-0.5*elbow_length} ${elbow_length - elbow_width} 0" rpy = "0 0 ${-pi/2}"/>
 			<geometry>
 				<box size = "${elbow_width} ${elbow_length} ${elbow_height}"/>
 			</geometry>
 		</visual>
-		<collision name = "elbow_link_collision">
-			<origin xyz = "${base_radius} ${base_radius} ${-mount_height}"/>
+		<collision name = "elbow_link_collsion">
+			<origin xyz = "${-mount_width/2} ${mount_length} 0" />
+			<geometry>
+				<box size = "${elbow_width} ${elbow_length} ${elbow_height}"/>
+			</geometry>
+		</collision>
+		<collision name = "second_elbow_link_collision">
+			<origin xyz = "${-0.5*elbow_length} ${elbow_length - elbow_width} 0" rpy = "0 0 ${-pi/2}"/>
 			<geometry>
 				<box size = "${elbow_width} ${elbow_length} ${elbow_height}"/>
@@ -94,5 +100,5 @@
 		<parent link = "mount_link" />
 		<child link = "elbow_link" />
-		<origin xyz = "${base_radius} ${base_radius} ${-mount_length}"/>
+		<origin xyz = "${base_radius} 0 ${-mount_height+elbow_height/2+base_height/2}" rpy="0 0 0"/>
 		<axis xyz = "1 0 0" />
 		<limit lower="${-pi/4}" upper="${pi/4}" effort="1000.0" velocity="10.0"/>
@@ -108,3 +114,29 @@
 		<origin xyz = "0 0 1" rpy = "0 0 0"/>
 	</joint>
+	<transmission name="pitch_transmission">
+		<type>transmission_interface/SimpleTransmission</type>
+		<joint name="pitch_joint">
+			<hardwareInterface>hardware_interface/PositionJointInterface</hardwareInterface>
+		</joint>
+		<actuator name="pitch_motor">
+			<hardwareInterface>hardware_interface/PositionJointInterface</hardwareInterface>
+			<mechanicalReduction>1</mechanicalReduction>
+		</actuator>
+	</transmission>
+	<transmission name="yaw_transmission">
+		<type>transmission_interface/SimpleTransmission</type>
+		<joint name="yaw_joint">
+			<hardwareInterface>hardware_interface/PositionJointInterface</hardwareInterface>
+		</joint>
+		<actuator name="yaw_motor">
+			<hardwareInterface>hardware_interface/PositionJointInterface</hardwareInterface>
+			<mechanicalReduction>1</mechanicalReduction>
+		</actuator>
+	</transmission>
+	<gazebo>
+		<static>false</static>
+		<plugin name = "gazebo_ros_control" filename = "libgazebo_ros_control.so">
+			<robotNamespace>/model</robotNamespace>
+		</plugin>
+	</gazebo>
 </robot>

Commit message: Added cylinder for scope, need to adjust joint and add mesh

File: urdf/model.urdf.xacro (robot description, xacro)
@@ -12,4 +12,7 @@
 	<xacro:property name = "elbow_height" value = "0.05"/>
 	<xacro:property name = "elbow_length" value = "0.15"/>
+	<xacro:property name = "scope_mass" value = "0.1"/>
+	<xacro:property name = "scope_length" value = "0.1"/>
+	<xacro:property name = "scope_radius" value = "0.015"/>
 	<link name = "world"/>
 	<link name = "base_link">
@@ -97,4 +100,35 @@
 		</collision>
 	</link>
+	<link name = "scope_link">
+		<inertial>
+			<mass value = "${scope_mass}"/>
+				<origin xyz = "${mount_length} 0 0 "/>
+			<inertia ixx = "0.0"
+					 ixy = "0.0"
+					 ixz = "0.0"
+					 iyy = "0.0"
+					 iyz = "0.0"
+					 izz = "0.0"/>
+			</inertial>
+		<visual name = "scope_link_visual">
+			<origin xyz = "${-mount_width/2} -${mount_length-mount_width} 0" rpy = "${pi/2} 0 0" />
+			<geometry>
+				<cylinder length = "${scope_length}" radius = "${scope_radius}"/>
+			</geometry>
+		</visual>
+		<collision name = "scope_link_collision">
+			<origin xyz = "${-mount_width/2} -${mount_length-mount_width} 0" rpy = "${pi/2} 0 0" />
+			<geometry>
+				<cylinder length = "${scope_length}" radius = "${scope_radius}"/>
+			</geometry>
+		</collision>
+	</link>
+	<joint name = "roll_joint" type = "revolute">
+		<parent link = "elbow_link" />
+		<child link = "scope_link" />
+		<origin xyz = "${-base_radius} ${base_radius} 0" rpy="0 0 0"/>
+		<axis xyz = "0 1 1" />
+		<limit lower="${-pi/4}" upper="${pi/4}" effort="1000.0" velocity="10.0"/>
+	</joint>
 	<joint name = "pitch_joint" type = "revolute">
 		<parent link = "mount_link" />
@@ -134,4 +168,14 @@
 		</actuator>
 	</transmission>
+	<transmission name="roll_transmission">
+		<type>transmission_interface/SimpleTransmission</type>
+		<joint name="roll_joint">
+			<hardwareInterface>hardware_interface/PositionJointInterface</hardwareInterface>
+		</joint>
+		<actuator name="roll_motor">
+			<hardwareInterface>hardware_interface/PositionJointInterface</hardwareInterface>
+			<mechanicalReduction>1</mechanicalReduction>
+		</actuator>
+	</transmission>
 	<gazebo>
 		<static>false</static>

Commit message: Using mesh for L-arm

File: urdf/model.urdf.xacro (robot description, xacro)
@@ -13,8 +13,8 @@
 	<xacro:property name = "elbow_length" value = "0.15"/>
 	<link name = "world"/>
-	<link name = "base_link">
-		<inertial>
-			<mass value = "${base_mass}"/>
-			<origin xyz = "0 0 0" rpy = "0 0 0"/>
+	<!--link name = "dummy_yaw_link">
+		<inertial>
+			<mass value="0.1"/>
+			<origin xyz="0 0 0" rpy="0 0 0"/>
 			<inertia ixx = "0.0"
 				 	 ixy = "0.0"
@@ -22,5 +22,29 @@
 				  	 iyy = "0.0"
 				 	 iyz = "0.0"
-				  	 izz="0.0"/>
+				  	 izz = "0.0"/>
+		</inertial>
+	</link>
+	<link name = "dummy_pitch_link">
+		<inertial>
+			<mass value="0.1"/>
+			<origin xyz="0 0 0" rpy="0 0 0"/>
+			<inertia ixx = "0.0"
+				 	 ixy = "0.0"
+				 	 ixz = "0.0"
+				  	 iyy = "0.0"
+				 	 iyz = "0.0"
+				  	 izz = "0.0"/>
+		</inertial>
+	</link-->
+	<link name = "base_link">
+		<inertial>
+			<mass value = "${base_mass}"/>
+			<origin xyz = "0 0 0" rpy = "0 0 0"/>
+			<inertia ixx = "0.0"
+				 	 ixy = "0.0"
+				 	 ixz = "0.0"
+				  	 iyy = "0.0"
+				 	 iyz = "0.0"
+				  	 izz = "0.0"/>
 		</inertial>
 		<visual name = "base_link_visual">
@@ -72,5 +96,5 @@
 					 izz = "0.0"/>
 			</inertial>
-		<visual name = "elbow_link_visual">
+		<!--visual name = "elbow_link_visual">
 			<origin xyz = "${-mount_width/2} ${mount_length} 0" />
 			<geometry>
@@ -83,4 +107,10 @@
 				<box size = "${elbow_width} ${elbow_length} ${elbow_height}"/>
 			</geometry>
+		</visual-->
+		<visual name = "elbow_link_visual">
+			<origin xyz = "${-mount_width/2} ${mount_length} 0" rpy="${pi} ${-pi/2} ${pi}"/>
+			<geometry>
+				<mesh filename="package://ysa_telescope/mesh/scope_arms_printable.STL" scale="0.001 0.001 0.001"/>
+			</geometry>
 		</visual>
 		<collision name = "elbow_link_collsion">
@@ -97,4 +127,24 @@
 		</collision>
 	</link>
+	<!--joint name="base_yaw_joint" type="continuous">
+		<parent link="world"/>
+		<child link="dummy_yaw_link"/>
+		<origin xyz = "0 0 1" rpy = "0 0 0"/>
+	</joint>
+	<joint name="base_pitch_joint" type="continuous">
+		<parent link="dummy_yaw_link"/>
+		<child link="dummy_pitch_link"/>
+		<origin xyz = "1 0 0" rpy = "0 0 0"/>
+	</joint-->
+	<joint name="fixed_link" type="fixed">
+		<parent link="world"/>
+		<child link="base_link"/>
+		<origin xyz="0 0 1"/>
+	</joint>
+	<joint name = "yaw_joint" type = "continuous">
+		<parent link = "base_link" />
+		<child link = "mount_link" />
+		<axis xyz = "0 0 1" />
+	</joint>
 	<joint name = "pitch_joint" type = "revolute">
 		<parent link = "mount_link" />
@@ -104,14 +154,4 @@
 		<limit lower="${-pi/4}" upper="${pi/4}" effort="1000.0" velocity="10.0"/>
 	</joint>
-	<joint name = "yaw_joint" type = "continuous">
-		<parent link = "base_link" />
-		<child link = "mount_link" />
-		<axis xyz = "0 0 1" />
-	</joint>
-	<joint name="world_joint" type="fixed">
-		<parent link="world"/>
-		<child link="base_link"/>
-		<origin xyz = "0 0 1" rpy = "0 0 0"/>
-	</joint>
 	<transmission name="pitch_transmission">
 		<type>transmission_interface/SimpleTransmission</type>
@@ -134,4 +174,24 @@
 		</actuator>
 	</transmission>
+	<!--transmission name="base_pitch_transmission">
+		<type>transmission_interface/SimpleTransmission</type>
+		<joint name="base_pitch_joint">
+			<hardwareInterface>hardware_interface/PositionJointInterface</hardwareInterface>
+		</joint>
+		<actuator name="base_pitch_motor">
+			<hardwareInterface>hardware_interface/PositionJointInterface</hardwareInterface>
+			<mechanicalReduction>1</mechanicalReduction>
+		</actuator>
+	</transmission>
+	<transmission name="base_yaw_transmission">
+		<type>transmission_interface/SimpleTransmission</type>
+		<joint name="base_yaw_joint">
+			<hardwareInterface>hardware_interface/PositionJointInterface</hardwareInterface>
+		</joint>
+		<actuator name="base_yaw_motor">
+			<hardwareInterface>hardware_interface/PositionJointInterface</hardwareInterface>
+			<mechanicalReduction>1</mechanicalReduction>
+		</actuator>
+	</transmission-->
 	<gazebo>
 		<static>false</static>

Commit message: Made small adjustments to joint location

File: urdf/model.urdf.xacro (robot description, xacro)
@@ -13,6 +13,6 @@
 	<xacro:property name = "elbow_length" value = "0.15"/>
 	<xacro:property name = "scope_mass" value = "0.1"/>
-	<xacro:property name = "scope_length" value = "0.1"/>
-	<xacro:property name = "scope_radius" value = "0.015"/>
+	<xacro:property name = "scope_length" value = "0.15"/>
+	<xacro:property name = "scope_radius" value = "0.02"/>
 	<link name = "world"/>
 	<!--link name = "dummy_yaw_link">
@@ -99,5 +99,5 @@
 					 izz = "0.0"/>
 			</inertial>
-		<!--visual name = "elbow_link_visual">
+		<visual name = "elbow_link_visual">
 			<origin xyz = "${-mount_width/2} ${mount_length} 0" />
 			<geometry>
@@ -110,11 +110,11 @@
 				<box size = "${elbow_width} ${elbow_length} ${elbow_height}"/>
 			</geometry>
+		</visual>
+		<!--visual name = "elbow_link_visual">
+			<origin xyz = "${-mount_width/2} ${mount_length} 0" rpy="${pi} ${-pi/2} ${pi}"/>
+			<geometry>
+				<mesh filename="package://ysa_telescope/mesh/scope_arms_printable.STL" scale="0.001 0.001 0.001"/>
+			</geometry>
 		</visual-->
-		<visual name = "elbow_link_visual">
-			<origin xyz = "${-mount_width/2} ${mount_length} 0" rpy="${pi} ${-pi/2} ${pi}"/>
-			<geometry>
-				<mesh filename="package://ysa_telescope/mesh/scope_arms_printable.STL" scale="0.001 0.001 0.001"/>
-			</geometry>
-		</visual>
 		<collision name = "elbow_link_collsion">
 			<origin xyz = "${-mount_width/2} ${mount_length} 0" />
@@ -133,5 +133,5 @@
 		<inertial>
 			<mass value = "${scope_mass}"/>
-				<origin xyz = "${mount_length} 0 0 "/>
+			<origin xyz = "${mount_length} 0 0 "/>
 			<inertia ixx = "0.0"
 					 ixy = "0.0"
@@ -142,5 +142,5 @@
 			</inertial>
 		<visual name = "scope_link_visual">
-			<origin xyz = "${-mount_width/2} -${mount_length-mount_width} 0" rpy = "${pi/2} 0 0" />
+			<origin xyz = "0 ${-scope_length/2} 0" rpy = "${pi/2} 0 0" />
 			<geometry>
 				<cylinder length = "${scope_length}" radius = "${scope_radius}"/>
@@ -148,5 +148,5 @@
 		</visual>
 		<collision name = "scope_link_collision">
-			<origin xyz = "${-mount_width/2} -${mount_length-mount_width} 0" rpy = "${pi/2} 0 0" />
+			<origin xyz = "0 ${-scope_length/2} 0" rpy = "${pi/2} 0 0" />
 			<geometry>
 				<cylinder length = "${scope_length}" radius = "${scope_radius}"/>
@@ -172,6 +172,6 @@
 		<parent link = "elbow_link" />
 		<child link = "scope_link" />
-		<origin xyz = "${-base_radius} ${base_radius} 0" rpy="0 0 0"/>
-		<axis xyz = "0 1 1" />
+		<origin xyz = "${-base_radius} ${elbow_length-elbow_width-mount_width/2} 0" rpy="0 0 0"/>
+		<axis xyz = "0 -1 0" />
 		<limit lower="${-pi/4}" upper="${pi/4}" effort="1000.0" velocity="10.0"/>
 	</joint>
@@ -188,11 +188,4 @@
 		<axis xyz = "0 0 1" />
 	</joint>
-	<joint name = "pitch_joint" type = "revolute">
-		<parent link = "mount_link" />
-		<child link = "elbow_link" />
-		<origin xyz = "${base_radius} 0 ${-mount_height+elbow_height/2+base_height/2}" rpy="0 0 0"/>
-		<axis xyz = "1 0 0" />
-		<limit lower="${-pi/4}" upper="${pi/4}" effort="1000.0" velocity="10.0"/>
-	</joint>
 	<transmission name="pitch_transmission">
 		<type>transmission_interface/SimpleTransmission</type>
@@ -211,4 +204,14 @@
 		</joint>
 		<actuator name="yaw_motor">
+			<hardwareInterface>hardware_interface/PositionJointInterface</hardwareInterface>
+			<mechanicalReduction>1</mechanicalReduction>
+		</actuator>
+	</transmission>
+	<transmission name="roll_transmission">
+		<type>transmission_interface/SimpleTransmission</type>
+		<joint name="roll_joint">
+			<hardwareInterface>hardware_interface/PositionJointInterface</hardwareInterface>
+		</joint>
+		<actuator name="roll_motor">
 			<hardwareInterface>hardware_interface/PositionJointInterface</hardwareInterface>
 			<mechanicalReduction>1</mechanicalReduction>
